Commit message: wip

File: test/single_joint.urdf (robot description, URDF)
Before this commit: robot single_joint, 2 links, 1 joints
Joints:
- removed joint joint
- added joint joint1: type revolute, parent base_link, child link1, origin xyz=0.2 0.01 0 rpy=0 0 0, axis 0 0 1, limit lower=-6.28 upper=6.28 effort=1000.0 velocity=0.5

Commit message: Working controller for simple set-up with a motor and encoder

File: test/single_joint.urdf (robot description, URDF)
Before this commit: robot single_joint, 2 links, 1 joints
Joints:
- joint joint1: limit lower=-6.28 upper=6.28 effort=1000.0 velocity=0.5 -> effort=1000.0 velocity=0.5; origin xyz=0.2 0.01 0 rpy=0 0 0 -> xyz=0.2 0.0 0 rpy=0 0 0; type revolute -> continuous
