Commit message: load full arm except for hand

File: test/sergio_arm.urdf (robot description, URDF)
Before this commit: robot sergio_arm, 2 links, 1 joints
Links:
- added link elbow_link4
- added link fore_arm
- added link shoulder_link1
- added link shoulder_mount
Joints:
- added joint elbow_pitch_joint: type revolute, parent upper_arm, child elbow_link4, origin xyz=0.01 -0.32 0.0 rpy=-1.5708 0 0, axis 0 -1 0, limit lower=0.0 upper=2.23 effort=4.5 velocity=1.0
- added joint elbow_roll_joint: type revolute, parent elbow_link4, child fore_arm, origin xyz=0.0 0.0 0.0 rpy=1.5708 0 0, axis 0 1 0, limit lower=-1.83 upper=1.83 effort=4.5 velocity=1.0
- added joint shoulder_pitch_joint: type revolute, parent shoulder_link1, child shoulder_link2, origin xyz=0.0 0.0 0.0 rpy=-1.5708  0 0, axis 0 -1 0, limit lower=-1.57 upper=1.57 effort=13.4 velocity=1.0
- added joint shoulder_yaw_joint: type revolute, parent shoulder_mount, child shoulder_link1, origin xyz=0 0 0 rpy=-1.5708 -1.5708 0, axis 1 0 0, limit lower=-1.57 upper=0.0 effort=13.4 velocity=1.0

Commit message: started on sergio hw iface

File: test/sergio_arm.urdf (robot description, URDF)
Before this commit: robot sergio_arm, 6 links, 5 joints
Links:
- removed link elbow_link4
- removed link fore_arm
- removed link upper_arm
- added link base_link
Joints:
- removed joint elbow_pitch_joint
- removed joint elbow_roll_joint
- removed joint shoulder_roll_joint
- added joint base_link_shoulder_joint: type fixed, parent base_link, child shoulder_mount, origin xyz=0 0.4 0 rpy=1.57 0 1.57

Commit message: Revert "started on sergio hw iface"
This reverts commit ad4de1723bb0c1553027b1a1935b286652457d63.

File: test/sergio_arm.urdf (robot description, URDF)
Before this commit: robot sergio_arm, 4 links, 3 joints
Links:
- removed link base_link
- added link elbow_link4
- added link fore_arm
- added link upper_arm
Joints:
- removed joint base_link_shoulder_joint
- added joint elbow_pitch_joint: type revolute, parent upper_arm, child elbow_link4, origin xyz=0.01 -0.32 0.0 rpy=-1.5708 0 0, axis 0 -1 0, limit lower=0.0 upper=2.23 effort=4.5 velocity=1.0
- added joint elbow_roll_joint: type revolute, parent elbow_link4, child fore_arm, origin xyz=0.0 0.0 0.0 rpy=1.5708 0 0, axis 0 1 0, limit lower=-1.83 upper=1.83 effort=4.5 velocity=1.0
- added joint shoulder_roll_joint: type revolute, parent shoulder_link2, child upper_arm, origin xyz=0.0 0.0 0.0 rpy=-1.5708  0 0, axis 0 -1 0, limit lower=-1.57 upper=1.57 effort=13.4 velocity=1.0

Commit message: param()Correct left arm representation

File: test/sergio_arm.urdf (robot description, URDF)
Before this commit: robot sergio_arm, 6 links, 5 joints
Links:
- added link base_link; visual box size=0.09 0.09 1.0
- added link torso; visual box size=0.09 0.6 0.09
- link fore_arm: geometry visual cylinder length=0.3 radius=0.05
- link upper_arm: geometry visual cylinder length=0.3 radius=0.05
Joints:
- added joint shoulder_mount_joint: type fixed, parent torso, child shoulder_mount, origin xyz=0.0 -0.3 0.0 rpy=0.0 0.0 0.0
- added joint torso_joint: type fixed, parent base_link, child torso, origin xyz=0.0 0.0 1.0 rpy=0.0 -1.57 3.1415
- joint elbow_roll_joint: axis 0 1 0 -> 0 -1 0
- joint shoulder_roll_joint: axis 0 -1 0 -> 0 1 0; origin xyz=0.0 0.0 0.0 rpy=-1.5708  0 0 -> xyz=0.0 0.0 0.0 rpy=1.5708  0 0

Commit message: Backup of athome12

File: test/sergio_arm.urdf (robot description, URDF)
Before this commit: robot sergio_arm, 8 links, 7 joints
Joints:
- joint shoulder_roll_joint: limit lower=-1.57 upper=1.57 effort=13.4 velocity=1.0 -> lower=-0.8 upper=0.8 effort=13.4 velocity=1.0
